File: STM32MCU.kicad_sch (KiCad schematic)
At the start: 13 parts, among them U1 PKU5511ESI, U5 STM32C542CCT6

Commit message: add footprints for standardized components
Parts:
- C6, C7, C8: footprint SOT-23-5_MC_MCH -> Capacitor_SMD:C_0603_1608Metric
- PS1, PS2, PS3, PS4: footprint E48SC12030NRFH -> (none)
- R11, R12, R13, R14: footprint E48SC12030NRFH -> Resistor_SMD:R_0603_1608Metric
- U1: footprint PKU5511ESI:CONV_PKU5511ESI -> (none)
- U5: footprint LQFP48-7X7 -> (none)
Changed lines of the file:
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@@
 			)
 		)
-		(property "Footprint" "LQFP48-7X7"
+		(property "Footprint" ""
 			(at 52.07 45.72 0)
 			(hide yes)
@@
 			)
 		)
-		(property "Footprint" "E48SC12030NRFH"
+		(property "Footprint" "Resistor_SMD:R_0603_1608Metric"
 			(at 246.126 144.526 90)
 			(hide yes)
@@
 			)
 		)
-		(property "Footprint" "SOT-23-5_MC_MCH"
+		(property "Footprint" "Capacitor_SMD:C_0603_1608Metric"
 			(at 127.3048 36.83 0)
 			(hide yes)
@@
 			)
 		)
-		(property "Footprint" "SOT-23-5_MC_MCH"
+		(property "Footprint" "Capacitor_SMD:C_0603_1608Metric"
 			(at 134.9248 67.31 0)
 			(hide yes)
@@
 			)
 		)
-		(property "Footprint" "SOT-23-5_MC_MCH"
+		(property "Footprint" "Capacitor_SMD:C_0603_1608Metric"
 			(at 43.4848 105.41 0)
 			(hide yes)
@@
 			)
 		)
-		(property "Footprint" "E48SC12030NRFH"
+		(property "Footprint" ""
 			(at 234.95 159.69 0)
 			(hide yes)
@@
 			)
 		)
-		(property "Footprint" "PKU5511ESI:CONV_PKU5511ESI"
+		(property "Footprint" ""
 			(at 85.09 162.56 0)
 			(hide yes)
@@
 			)
 		)
-		(property "Footprint" "E48SC12030NRFH"
+		(property "Footprint" ""
 			(at 234.95 129.21 0)
 			(hide yes)
@@
 			)
 		)
-		(property "Footprint" "E48SC12030NRFH"
+		(property "Footprint" "Resistor_SMD:R_0603_1608Metric"
 			(at 135.636 58.674 90)
 			(hide yes)
@@
 			)
 		)
-		(property "Footprint" "E48SC12030NRFH"
+		(property "Footprint" ""
 			(at 234.95 192.71 0)
 			(hide yes)
@@
 			)
 		)
-		(property "Footprint" "E48SC12030NRFH"
+		(property "Footprint" ""
 			(at 234.95 225.73 0)
 			(hide yes)
@@
 			)
 		)
-		(property "Footprint" "E48SC12030NRFH"
+		(property "Footprint" "Resistor_SMD:R_0603_1608Metric"
 			(at 247.396 78.486 90)
 			(hide yes)
@@
 			)
 		)
-		(property "Footprint" "E48SC12030NRFH"
+		(property "Footprint" "Resistor_SMD:R_0603_1608Metric"
 			(at 247.396 111.506 90)
 			(hide yes)
