File: X19-Power-Slab-Board.kicad_sch (KiCad schematic)
At the start: 43 parts, among them J1 Conn_01x03_Pin, J10 Conn_01x02, J11 Conn_01x02, J12 Conn_01x02, J13 Conn_01x02, J2 796636-6, J3 Conn_01x03_Pin, J4 Conn_01x04_Pin, J5 Conn_02x05_Odd_Even, J6 Conn_01x02, J7 Conn_01x02, J8 Conn_01x02, J9 Conn_01x02, U1 TCAN1044AEV-Q1, U2 TMP1075NDRLR

Commit message: Bennett TODOs
Other:
- note added: "100V Rated Electrolytic"
- note added: "CHANGES 1. find and implemeent footprint for 16MHz 2. any non power capacitors --> 0805 (default kicad) 3. LED resistor size 4. Find capacitors for bulk power stuff 5. change brick to I6A"
- note added: "~10mA thru each LED account for LED forward voltage drop"
Changed lines of the file:
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@@
+		)
+	)
+	(text "100V Rated\nElectrolytic\n"
+		(exclude_from_sim no)
+		(at 83.82 53.34 0)
+		(effects
+			(font
+				(size 1.27 1.27)
+				(color 255 43 0 1)
+			)
 		)
 	)
@@
 		)
 	)
+	(text "~10mA thru each LED\naccount for LED forward voltage drop"
+		(exclude_from_sim no)
+		(at 36.83 149.86 0)
+		(effects
+			(font
+				(size 1.27 1.27)
+				(color 255 0 19 1)
+			)
+		)
+	)
 	(text "CAN ESD Protection"
 		(exclude_from_sim no)
@@
 			)
 		)
+	)
+	(text "CHANGES\n1. find and implemeent footprint for 16MHz\n2. any non power capacitors --> 0805 (default kicad)\n3. LED resistor size\n4. Find capacitors for bulk power stuff\n5. change brick to I6A"
+		(exclude_from_sim no)
+		(at 220.98 147.32 0)
+		(effects
+			(font
+				(size 2.54 2.54)
+				(thickness 0.508)
+				(bold yes)
+				(color 255 13 0 1)
+			)
+		)

Commit message: updated some of nicks requested changes
Parts:
- removed 12V: RED, symbol Device:LED
- added D1: LED, i6A4W_DIP_FULL_TDK, symbol Device:LED
- J2: footprint CON6_P5MM_VER_TERM-BLK_TYC -> rov_connectors:CON6_P5MM_VER_TERM-BLK_TYC
- R1: value 330 -> 300
- R3: value 330 -> 120
- R4, R5: value 2.4k -> 2.2k
- U1: footprint D0008A-IPC_A -> rov_logic:D0008A-IPC_A
- U2: footprint SOT5X3-6_DRL_TEX -> rov_sensors:SOT5X3-6_DRL_TEX
- renumbered 3.3V to D3, 48V to D4, 5.1V to D5
Connections:
- net GND: now also D1.1 (K)
- net at R2.1: now also D1.2 (A)
Changed lines of the file:
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@@
 			)
 		)
-		(property "Footprint" "CON6_P5MM_VER_TERM-BLK_TYC"
+		(property "Footprint" "rov_connectors:CON6_P5MM_VER_TERM-BLK_TYC"
 			(at 35.56 81.28 0)
 			(hide yes)
@@
 			)
 		)
-		(property "Value" "330"
+		(property "Value" "300"
 			(at 26.67 130.8099 0)
 			(show_name no)
@@
 		(dnp no)
 		(fields_autoplaced yes)
-		(property "Reference" "3.3V"
+		(property "Reference" "D3"
 			(at 57.15 137.4774 90)
 			(show_name no)
@@
 			(project "X19-Power-Slab-Board"
 				(path "/00000000-0000-0000-0000-000060e6118b"
-					(reference "3.3V")
+					(reference "D3")
 					(unit 1)
 				)
@@
 	)
 	(symbol
+		(lib_id "Device:LED")
+		(at 39.37 137.16 90)
+		(unit 1)
+		(body_style 1)
+		(exclude_from_sim no)
+		(in_bom yes)
+		(on_board yes)
+		(in_pos_files yes)
+		(dnp no)
+		(fields_autoplaced yes)
+		(property "Reference" "D1"
+			(at 43.18 137.4774 90)
+			(show_name no)
+			(do_not_autoplace no)
+			(effects
+				(font
+					(size 1.27 1.27)
+				)
+				(justify right)
+			)
+		)
+		(property "Value" "LED"
+			(at 43.18 140.0174 90)
+			(show_name no)
+			(do_not_autoplace no)
+			(effects
+				(font
+					(size 1.27 1.27)
+				)
+				(justify right)
+			)
+		)
+		(property "Footprint" "i6A4W_DIP_FULL_TDK"
+			(at 39.37 137.16 0)
+			(hide yes)
+			(show_name no)
+			(do_not_autoplace no)
+			(effects
+				(font
+					(size 1.27 1.27)
+				)
+			)
+		)
+		(property "Datasheet" ""
+			(at 39.37 137.16 0)
+			(hide yes)
+			(show_name no)
+			(do_not_autoplace no)
+			(effects
+				(font
+					(size 1.27 1.27)
+				)
+			)
+		)
+		(property "Description" "Light emitting diode"
+			(at 39.37 137.16 0)
+			(hide yes)
+			(show_name no)
+			(do_not_autoplace no)
+			(effects
+				(font
+					(size 1.27 1.27)
+				)
+			)
+		)
+		(property "Sim.Pins" "1=K 2=A"
+			(at 39.37 137.16 0)
+			(hide yes)
+			(show_name no)
+			(do_not_autoplace no)
+			(effects
+				(font
+					(size 1.27 1.27)
+				)
+			)
+		)
+		(pin "2"
+		)
+		(pin "1"
+		)
+		(instances
+			(project "X19-Power-Slab-Board"
+				(path "/00000000-0000-0000-0000-000060e6118b"
+					(reference "D1")
+					(unit 1)
+				)
+			)
+		)
+	)
+	(symbol
 		(lib_id "power:+3V3")
 		(at 73.66 92.71 90)
@@
 			)
 		)
-		(property "Value" "330"
+		(property "Value" "120"
 			(at 55.88 130.8099 0)
 			(show_name no)
@@
 			)
 		)
-		(property "Value" "2.4k"
+		(property "Value" "2.2k"
 			(at 71.12 130.81 0)
 			(show_name no)
@@
 	)
 	(symbol
-		(lib_id "Device:LED")
-		(at 39.37 137.16 90)
-		(unit 1)
-		(body_style 1)
-		(exclude_from_sim no)
-		(in_bom yes)
-		(on_board yes)
-		(in_pos_files yes)
-		(dnp no)
-		(fields_autoplaced yes)
-		(property "Reference" "12V"
-			(at 43.18 137.4774 90)
-			(show_name no)
-			(do_not_autoplace no)
-			(effects
-				(font
-					(size 1.27 1.27)
-				)
-				(justify right)
-			)
-		)
-		(property "Value" "RED"
-			(at 43.18 140.0174 90)
-			(show_name no)
-			(do_not_autoplace no)
-			(effects
-				(font
-					(size 1.27 1.27)
-				)
-				(justify right)
-			)
-		)
-		(property "Footprint" ""
-			(at 39.37 137.16 0)
-			(hide yes)
-			(show_name no)
-			(do_not_autoplace no)
-			(effects
-				(font
-					(size 1.27 1.27)
-				)
-			)
-		)
-		(property "Datasheet" ""
-			(at 39.37 137.16 0)
-			(hide yes)
-			(show_name no)
-			(do_not_autoplace no)
-			(effects
-				(font
-					(size 1.27 1.27)
-				)
-			)
-		)
-		(property "Description" "Light emitting diode"
-			(at 39.37 137.16 0)
-			(hide yes)
-			(show_name no)
-			(do_not_autoplace no)
-			(effects
-				(font
-					(size 1.27 1.27)
-				)
-			)
-		)
-		(property "Sim.Pins" "1=K 2=A"
-			(at 39.37 137.16 0)
-			(hide yes)
-			(show_name no)
-			(do_not_autoplace no)
-			(effects
-				(font
-					(size 1.27 1.27)
-				)
-			)
-		)
-		(pin "1"
-		)
-		(pin "2"
-		)
-		(instances
-			(project "X19-Power-Slab-Board"
-				(path "/00000000-0000-0000-0000-000060e6118b"
-					(reference "12V")
-					(unit 1)
-				)
-			)
-		)
-	)
-	(symbol
 		(lib_id "Connector:TestPoint")
 		(at 100.33 171.45 180)
@@
 		(dnp no)
 		(fields_autoplaced yes)
-		(property "Reference" "48V"
+		(property "Reference" "D4"
 			(at 71.12 145.0974 90)
 			(show_name no)
@@
 			(project "X19-Power-Slab-Board"
 				(path "/00000000-0000-0000-0000-000060e6118b"
-					(reference "48V")
+					(reference "D4")
 					(unit 1)
 				)
@@
 			)
 		)
-		(property "Footprint" "SOT5X3-6_DRL_TEX"
+		(property "Footprint" "rov_sensors:SOT5X3-6_DRL_TEX"
 			(at 215.9 31.75 0)
 			(hide yes)
@@
 			)
 		)
-		(property "Footprint" "D0008A-IPC_A"
+		(property "Footprint" "rov_logic:D0008A-IPC_A"
 			(at 104.14 30.48 0)
 			(hide yes)
@@
 		(dnp no)
 		(fields_autoplaced yes)
-		(property "Reference" "5.1V"
+		(property "Reference" "D5"
 			(at 27.94 137.4774 90)
 			(show_name no)
@@
 			(project "X19-Power-Slab-Board"
 				(path "/00000000-0000-0000-0000-000060e6118b"
-					(reference "5.1V")
+					(reference "D5")
 					(unit 1)
 				)
@@
 			)
 		)
-		(property "Value" "2.4k"
+		(property "Value" "2.2k"
 			(at 71.12 138.43 0)
 			(show_name no)

Commit message: meeting notes and quick changes, someone needs to verify new components
Parts:
- removed D4: BLUE, symbol Device:LED
- removed R4, R5: 2.2k, symbol Device:R_US
Other:
- note added: "resistros 0603, led 0805"

Commit message: assigned some cap and res footprints
Parts:
- C3: footprint (none) -> Capacitor_SMD:C_1206_3216Metric_Pad1.33x1.80mm_HandSolder
- C4, C44, C5, C6: footprint (none) -> Capacitor_SMD:C_0603_1608Metric_Pad1.08x0.95mm_HandSolder
- D1: footprint i6A4W_DIP_FULL_TDK -> LED_SMD:LED_0805_2012Metric_Pad1.15x1.40mm_HandSolder
- D3, D5: footprint (none) -> LED_SMD:LED_0805_2012Metric_Pad1.15x1.40mm_HandSolder
- J1, J3: footprint (none) -> Connector_PinHeader_2.54mm:PinHeader_1x03_P2.54mm_Vertical
- J10, J11, J12, J13, J6, J7, J8, J9: footprint (none) -> Connector_PinHeader_2.54mm:PinHeader_1x02_P2.54mm_Vertical
- J4: footprint (none) -> Connector_PinHeader_2.54mm:PinHeader_1x04_P2.54mm_Vertical
- J5: footprint (none) -> Connector_PinHeader_2.54mm:PinHeader_2x05_P2.54mm_Vertical
- R1, R2, R25, R26, R3, R6: footprint (none) -> Resistor_SMD:R_0603_1608Metric_Pad0.98x0.95mm_HandSolder
- TP6, TP7: footprint (none) -> TestPoint:TestPoint_Pad_D4.0mm
Changed lines of the file:
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@@
 			)
 		)
-		(property "Footprint" ""
+		(property "Footprint" "Connector_PinHeader_2.54mm:PinHeader_1x04_P2.54mm_Vertical"
 			(at 49.53 189.23 0)
 			(hide yes)
@@
 			)
 		)
-		(property "Footprint" ""
+		(property "Footprint" "Capacitor_SMD:C_0603_1608Metric_Pad1.08x0.95mm_HandSolder"
 			(at 186.9948 43.18 0)
 			(hide yes)
@@
 			)
 		)
-		(property "Footprint" ""
+		(property "Footprint" "Connector_PinHeader_2.54mm:PinHeader_1x02_P2.54mm_Vertical"
 			(at 265.43 81.28 0)
 			(hide yes)
@@
 			)
 		)
-		(property "Footprint" ""
+		(property "Footprint" "Resistor_SMD:R_0603_1608Metric_Pad0.98x0.95mm_HandSolder"
 			(at 38.354 129.286 90)
 			(hide yes)
@@
 			)
 		)
-		(property "Footprint" ""
+		(property "Footprint" "Connector_PinHeader_2.54mm:PinHeader_1x03_P2.54mm_Vertical"
 			(at 48.26 170.18 0)
 			(hide yes)
@@
 			)
 		)
-		(property "Footprint" ""
+		(property "Footprint" "Capacitor_SMD:C_0603_1608Metric_Pad1.08x0.95mm_HandSolder"
 			(at 275.8948 38.1 0)
 			(hide yes)
@@
 			)
 		)
-		(property "Footprint" ""
+		(property "Footprint" "Connector_PinHeader_2.54mm:PinHeader_1x02_P2.54mm_Vertical"
 			(at 265.43 63.5 0)
 			(hide yes)
@@
 			)
 		)
-		(property "Footprint" ""
+		(property "Footprint" "Resistor_SMD:R_0603_1608Metric_Pad0.98x0.95mm_HandSolder"
 			(at 23.114 129.286 90)
 			(hide yes)
@@
 			)
 		)
-		(property "Footprint" ""
+		(property "Footprint" "LED_SMD:LED_0805_2012Metric_Pad1.15x1.40mm_HandSolder"
 			(at 53.34 137.16 0)
 			(hide yes)
@@
 			)
 		)
-		(property "Footprint" ""
+		(property "Footprint" "Capacitor_SMD:C_0603_1608Metric_Pad1.08x0.95mm_HandSolder"
 			(at 158.75 38.4048 0)
 			(hide yes)
@@
 			)
 		)
-		(property "Footprint" ""
+		(property "Footprint" "Connector_PinHeader_2.54mm:PinHeader_1x03_P2.54mm_Vertical"
 			(at 31.75 170.18 0)
 			(hide yes)
@@
 			)
 		)
-		(property "Footprint" ""
+		(property "Footprint" "TestPoint:TestPoint_Pad_D4.0mm"
 			(at 139.7 81.28 0)
 			(hide yes)
@@
 			)
 		)
-		(property "Footprint" ""
+		(property "Footprint" "Connector_PinHeader_2.54mm:PinHeader_1x02_P2.54mm_Vertical"
 			(at 265.43 116.84 0)
 			(hide yes)
@@
 			)
 		)
-		(property "Footprint" "i6A4W_DIP_FULL_TDK"
+		(property "Footprint" "LED_SMD:LED_0805_2012Metric_Pad1.15x1.40mm_HandSolder"
 			(at 39.37 137.16 0)
 			(hide yes)
@@
 			)
 		)
-		(property "Footprint" ""
+		(property "Footprint" "Resistor_SMD:R_0603_1608Metric_Pad0.98x0.95mm_HandSolder"
 			(at 147.066 35.814 90)
 			(hide yes)
@@
 			)
 		)
-		(property "Footprint" ""
+		(property "Footprint" "Resistor_SMD:R_0603_1608Metric_Pad0.98x0.95mm_HandSolder"
 			(at 214.884 26.924 90)
 			(hide yes)
@@
 			)
 		)
-		(property "Footprint" ""
+		(property "Footprint" "Resistor_SMD:R_0603_1608Metric_Pad0.98x0.95mm_HandSolder"
 			(at 52.324 129.286 90)
 			(hide yes)
@@
 			)
 		)
-		(property "Footprint" ""
+		(property "Footprint" "Connector_PinHeader_2.54mm:PinHeader_1x02_P2.54mm_Vertical"
 			(at 265.43 72.39 0)
 			(hide yes)
@@
 			)
 		)
-		(property "Footprint" ""
+		(property "Footprint" "Resistor_SMD:R_0603_1608Metric_Pad0.98x0.95mm_HandSolder"
 			(at 147.066 43.434 90)
 			(hide yes)
@@
 			)
 		)
-		(property "Footprint" ""
+		(property "Footprint" "TestPoint:TestPoint_Pad_D4.0mm"
 			(at 129.54 83.82 0)
 			(hide yes)
@@
 			)
 		)
-		(property "Footprint" ""
+		(property "Footprint" "Connector_PinHeader_2.54mm:PinHeader_1x02_P2.54mm_Vertical"
 			(at 265.43 90.17 0)
 			(hide yes)
@@
 			)
 		)
-		(property "Footprint" ""
+		(property "Footprint" "Connector_PinHeader_2.54mm:PinHeader_2x05_P2.54mm_Vertical"
 			(at 78.74 87.63 0)
 			(hide yes)
@@
 			)
 		)
-		(property "Footprint" ""
+		(property "Footprint" "Capacitor_SMD:C_0603_1608Metric_Pad1.08x0.95mm_HandSolder"
 			(at 173.0248 43.18 0)
 			(hide yes)
@@
 			)
 		)
-		(property "Footprint" ""
+		(property "Footprint" "Connector_PinHeader_2.54mm:PinHeader_1x02_P2.54mm_Vertical"
 			(at 265.43 107.95 0)
 			(hide yes)
@@
 			)
 		)
-		(property "Footprint" ""
+		(property "Footprint" "Connector_PinHeader_2.54mm:PinHeader_1x02_P2.54mm_Vertical"
 			(at 265.43 125.73 0)
 			(hide yes)
@@
 			)
 		)
-		(property "Footprint" ""
+		(property "Footprint" "LED_SMD:LED_0805_2012Metric_Pad1.15x1.40mm_HandSolder"
 			(at 24.13 137.16 0)
 			(hide yes)
@@
 			)
 		)
-		(property "Footprint" ""
+		(property "Footprint" "Connector_PinHeader_2.54mm:PinHeader_1x02_P2.54mm_Vertical"
 			(at 265.43 99.06 0)
 			(hide yes)
@@
 			)
 		)
-		(property "Footprint" ""
+		(property "Footprint" "Capacitor_SMD:C_1206_3216Metric_Pad1.33x1.80mm_HandSolder"
 			(at 68.2752 40.64 0)
 			(hide yes)

Commit message: office hour changes
Parts:
- 12V1, 48V1: footprint Package_SO:SOIC-24W_7.5x15.4mm_P1.27mm -> TestPoint:TestPoint_Pad_D4.0mm
- 3.3V1, 5.1V1: footprint Package_SO:SOIC-24W_7.5x15.4mm_P1.27mm -> TestPoint:TestPoint_Pad_D2.5mm
- C1, C2: footprint (none) -> Capacitor_THT:CP_Radial_D13.0mm_P5.00mm
- CR2: footprint SOT-23_DBZ_TEX -> Package_TO_SOT_SMD:SOT-23_Handsoldering
Changed lines of the file:
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@@
 			)
 		)
-		(property "Footprint" "Package_SO:SOIC-24W_7.5x15.4mm_P1.27mm"
+		(property "Footprint" "TestPoint:TestPoint_Pad_D2.5mm"
 			(at 114.3 171.45 0)
 			(hide yes)
@@
 			)
 		)
-		(property "Footprint" ""
+		(property "Footprint" "Capacitor_THT:CP_Radial_D13.0mm_P5.00mm"
 			(at 50.8 36.83 0)
 			(hide yes)
@@
 			)
 		)
-		(property "Footprint" "Package_SO:SOIC-24W_7.5x15.4mm_P1.27mm"
+		(property "Footprint" "TestPoint:TestPoint_Pad_D2.5mm"
 			(at 83.82 171.45 0)
 			(hide yes)
@@
 			)
 		)
-		(property "Footprint" "Package_SO:SOIC-24W_7.5x15.4mm_P1.27mm"
+		(property "Footprint" "TestPoint:TestPoint_Pad_D4.0mm"
 			(at 95.25 171.45 0)
 			(hide yes)
@@
 			)
 		)
-		(property "Footprint" ""
+		(property "Footprint" "Capacitor_THT:CP_Radial_D13.0mm_P5.00mm"
 			(at 35.56 36.83 0)
 			(hide yes)
@@
 			)
 		)
-		(property "Footprint" "Package_SO:SOIC-24W_7.5x15.4mm_P1.27mm"
+		(property "Footprint" "TestPoint:TestPoint_Pad_D4.0mm"
 			(at 72.39 171.45 0)
 			(hide yes)
@@
 			)
 		)
-		(property "Footprint" "SOT-23_DBZ_TEX"
+		(property "Footprint" "Package_TO_SOT_SMD:SOT-23_Handsoldering"
 			(at 130.556 89.916 0)
 			(hide yes)
