File: power.kicad_sch (KiCad schematic)
At the start: 45 parts, among them U4 MIC5504-3.3YM5-TR

Commit message: updated some of nicks requested changes
Parts:
- removed PS1: IRS-5_10-Q12P-C, IRS510Q12PC, symbol IRS-5_10-Q12P-C:IRS-5_10-Q12P-C
- added R28: 10k, symbol Device:R_US
- added U7: i6A4W020A033V-003-R, i6A4W_DIP_FULL_TDK, symbol 2026-10-14_21-27-49:i6A4W020A033V-003-R
- B2, B3, B4, B5: footprint E48SC12030NRFH -> rov_power:E48SC12030NRFH
- C17, C21, U4: footprint SOT-23-5_MC_MCH -> rov_power:SOT-23-5_MC_MCH
- C19: value 1uF -> 0.1uF
- C20: value 470uF -> 22uF
Connections:
- net +3.3V: now also R28.1
- net +48V: now also U7.1 (VIN(+))
- net +5.1V_RAW: now also U7.7 (SENSE(+)), U7.8 (VOUT(+)); no longer R27.2
- net 48V_RETURN: now also U7.3 (VIN(-))
- net GND: now also R27.2, U7.4 (VOUT(-))
- net at R27.1: now also U7.6 (TRIM)
- new net: R28.2, U7.34 (SEQ)
Other:
- moved on the sheet: C16, C18, C19, C20, R27

Commit message: meeting notes and quick changes, someone needs to verify new components
Other:
- note added: "25V for right 63V for left 22uF 1206, 0603 for <1uF, custom for 100"
- note added: "63V 1206 caps"
- note added: "Can drop down to 63V, ideally would be 100V keep 63V if its too big (USE 63V)"
- note added: "Low ESR 63V (VIN+/VIN-)"
- note added: "Low ESR 63V Electrolytic (VIN+/VIN-)"
- note removed: "100V X7R"
- note removed: "10V X7R"
- note removed: "Can drop down to 63V, ideally would be 100V keep 63V if its too big"
- note removed: "Datasheet specifies >330uF output capacitance between OUT+, OUT-"
- note removed: "Low ESR 100V (VIN+/VIN-)"
- note removed: "Low ESR 100V Electrolytic (VIN+/VIN-)"
- note removed: "Low ESR Input 100V Rated"
- note removed: "R value From Datasheet pg. 36"
Changed lines of the file:
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@@
 		)
 	)
-	(text "Datasheet specifies\n>330uF output capacitance\nbetween OUT+, OUT-"
-		(exclude_from_sim no)
-		(at 80.01 124.46 0)
+	(text "3.3V LDO"
+		(exclude_from_sim no)
+		(at 19.558 22.86 0)
+		(effects
+			(font
+				(size 1.27 1.27)
+			)
+		)
+	)
+	(text "CHECK CAPACITORS \nCHECK DATASHEET OF I6A\nTO SEE WHAT MINIMUM OUPTUT"
+		(exclude_from_sim no)
+		(at 53.34 150.114 0)
+		(effects
+			(font
+				(size 1.27 1.27)
+				(color 255 37 1 1)
+			)
+		)
+	)
+	(text "360W Bricks 48V - 12V (4x)"
+		(exclude_from_sim no)
+		(at 190.5 22.606 0)
+		(effects
+			(font
+				(size 1.27 1.27)
+			)
+		)
+	)
+	(text "Brick Passives"
+		(exclude_from_sim no)
+		(at 104.14 22.86 0)
+		(effects
+			(font
+				(size 1.27 1.27)
+			)
+		)
+	)
+	(text "Low ESR 63V \n(VIN+/VIN-)"
+		(exclude_from_sim no)
+		(at 106.68 53.34 0)
+		(effects
+			(font
+				(size 1.27 1.27)
+			)
+		)
+	)
+	(text "50W Brick 48V - 5.1V"
+		(exclude_from_sim no)
+		(at 25.654 61.976 0)
+		(effects
+			(font
+				(size 1.27 1.27)
+			)
+		)
+	)
+	(text "Use 25V Rated Cap\n"
+		(exclude_from_sim no)
+		(at 82.55 137.16 0)
+		(effects
+			(font
+				(size 1.27 1.27)
+			)
+		)
+	)
+	(text "OUTPUT"
+		(exclude_from_sim no)
+		(at 77.47 116.84 0)
+		(effects
+			(font
+				(size 1.27 1.27)
+			)
+		)
+	)
+	(text "INPUT"
+		(exclude_from_sim no)
+		(at 29.21 116.84 0)
+		(effects
+			(font
+				(size 1.27 1.27)
+			)
+		)
+	)
+	(text "I2C Address: \n0x21 (Hex)"
+		(exclude_from_sim no)
+		(at 267.97 77.47 0)
+		(effects
+			(font
+				(size 1.27 1.27)
+			)
+		)
+	)
+	(text "Low ESR 63V\nElectrolytic \n(VIN+/VIN-)"
+		(exclude_from_sim no)
+		(at 106.68 34.29 0)
+		(effects
+			(font
+				(size 1.27 1.27)
+			)
+		)
+	)
+	(text ""
+		(exclude_from_sim no)
+		(at 55.118 132.842 0)
 		(effects
 			(font
@@
 		)
 	)
-	(text "3.3V LDO"
-		(exclude_from_sim no)
-		(at 19.558 22.86 0)
-		(effects
-			(font
-				(size 1.27 1.27)
-			)
-		)
-	)
-	(text "CHECK CAPACITORS \nCHECK DATASHEET OF I6A\nTO SEE WHAT MINIMUM OUPTUT"
-		(exclude_from_sim no)
-		(at 53.34 150.114 0)
-		(effects
-			(font
-				(size 1.27 1.27)
-				(color 255 37 1 1)
-			)
-		)
-	)
-	(text "360W Bricks 48V - 12V (4x)"
-		(exclude_from_sim no)
-		(at 190.5 22.606 0)
-		(effects
-			(font
-				(size 1.27 1.27)
-			)
-		)
-	)
-	(text "Low ESR Input\n100V Rated"
-		(exclude_from_sim no)
-		(at 22.86 119.38 0)
-		(effects
-			(font
-				(size 0.635 0.635)
-			)
-		)
-	)
-	(text "Brick Passives"
-		(exclude_from_sim no)
-		(at 104.14 22.86 0)
-		(effects
-			(font
-				(size 1.27 1.27)
-			)
-		)
-	)
-	(text "Low ESR 100V \n(VIN+/VIN-)"
-		(exclude_from_sim no)
-		(at 106.68 53.34 0)
-		(effects
-			(font
-				(size 1.27 1.27)
-			)
-		)
-	)
-	(text "50W Brick 48V - 5.1V"
-		(exclude_from_sim no)
-		(at 25.654 61.976 0)
-		(effects
-			(font
-				(size 1.27 1.27)
-			)
-		)
-	)
-	(text "Use 25V Rated Cap\n"
-		(exclude_from_sim no)
-		(at 82.55 137.16 0)
-		(effects
-			(font
-				(size 1.27 1.27)
-			)
-		)
-	)
-	(text "OUTPUT"
-		(exclude_from_sim no)
-		(at 77.47 116.84 0)
-		(effects
-			(font
-				(size 1.27 1.27)
-			)
-		)
-	)
-	(text "INPUT"
-		(exclude_from_sim no)
-		(at 29.21 116.84 0)
-		(effects
-			(font
-				(size 1.27 1.27)
-			)
-		)
-	)
-	(text "I2C Address: \n0x21 (Hex)"
-		(exclude_from_sim no)
-		(at 267.97 77.47 0)
-		(effects
-			(font
-				(size 1.27 1.27)
-			)
-		)
-	)
-	(text "Low ESR 100V\nElectrolytic \n(VIN+/VIN-)"
-		(exclude_from_sim no)
-		(at 106.68 34.29 0)
-		(effects
-			(font
-				(size 1.27 1.27)
-			)
-		)
-	)
-	(text ""
-		(exclude_from_sim no)
-		(at 55.118 132.842 0)
-		(effects
-			(font
-				(size 0.635 0.635)
+	(text "63V 1206 caps"
+		(exclude_from_sim no)
+		(at 165.1 58.674 0)
+		(effects
+			(font
+				(size 1.27 1.27)
+				(color 255 0 23 1)
 			)
 		)
@@
 		)
 	)
-	(text "10V X7R"
-		(exclude_from_sim no)
-		(at 67.31 119.38 0)
-		(effects
-			(font
-				(size 0.635 0.635)
-			)
-		)
-	)
 	(text "INPUT"
 		(exclude_from_sim no)
@@
 		)
 	)
+	(text "25V for right\n63V for left\n22uF 1206, 0603 for <1uF, custom for 100\n"
+		(exclude_from_sim no)
+		(at 47.244 139.192 0)
+		(effects
+			(font
+				(size 1.27 1.27)
+				(color 255 5 28 1)
+			)
+		)
+	)
 	(text "BRICK SHOULD BE THIS\nI6A4W020A033V-003-R"
 		(exclude_from_sim no)
@@
 		)
 	)
-	(text "R value\nFrom Datasheet pg. 36"
-		(exclude_from_sim no)
-		(at 52.578 132.842 0)
-		(effects
-			(font
-				(size 0.635 0.635)
-			)
-		)
-	)
 	(text "I2C Address: \n0x22 (Hex)"
 		(exclude_from_sim no)
@@
 		)
 	)
-	(text "Can drop down to 63V,\nideally would be 100V\nkeep 63V if its too big"
+	(text "Can drop down to 63V,\nideally would be 100V\nkeep 63V if its too big\n(USE 63V)\n"
 		(exclude_from_sim no)
 		(at 147.32 44.45 0)
@@
 			)
 		)
-	)
-	(text "100V X7R"
-		(exclude_from_sim no)
-		(at 35.56 125.73 0)
-		(effects
-			(font
-				(size 0.635 0.635)
-			)
-		)

Commit message: assigned some cap and res footprints
Parts:
- C17, C21: footprint rov_power:SOT-23-5_MC_MCH -> Capacitor_SMD:C_0603_1608Metric_Pad1.08x0.95mm_HandSolder
- C18, C19, C26, C31, C33, C38: footprint (none) -> Capacitor_SMD:C_0603_1608Metric_Pad1.08x0.95mm_HandSolder
- C20, C23, C27, C32, C37: footprint (none) -> Capacitor_SMD:C_1206_3216Metric_Pad1.33x1.80mm_HandSolder
- PG1, PG2, PG3, PG4: footprint (none) -> TestPoint:TestPoint_Pad_D4.0mm
- R13, R14, R15, R16, R17, R18, R19, R20, R27, R28: footprint (none) -> Resistor_SMD:R_0603_1608Metric_Pad0.98x0.95mm_HandSolder
Changed lines of the file:
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@@
 			)
 		)
-		(property "Footprint" ""
+		(property "Footprint" "Resistor_SMD:R_0603_1608Metric_Pad0.98x0.95mm_HandSolder"
 			(at 241.046 122.174 90)
 			(hide yes)
@@
 			)
 		)
-		(property "Footprint" ""
+		(property "Footprint" "Capacitor_SMD:C_0603_1608Metric_Pad1.08x0.95mm_HandSolder"
 			(at 157.1752 118.11 0)
 			(hide yes)
@@
 			)
 		)
-		(property "Footprint" ""
+		(property "Footprint" "Resistor_SMD:R_0603_1608Metric_Pad0.98x0.95mm_HandSolder"
 			(at 83.566 80.264 90)
 			(hide yes)
@@
 			)
 		)
-		(property "Footprint" ""
+		(property "Footprint" "TestPoint:TestPoint_Pad_D4.0mm"
 			(at 194.31 153.67 0)
 			(hide yes)
@@
 			)
 		)
-		(property "Footprint" ""
+		(property "Footprint" "Capacitor_SMD:C_0603_1608Metric_Pad1.08x0.95mm_HandSolder"
 			(at 68.2752 134.62 0)
 			(hide yes)
@@
 			)
 		)
-		(property "Footprint" ""
+		(property "Footprint" "Capacitor_SMD:C_1206_3216Metric_Pad1.33x1.80mm_HandSolder"
 			(at 79.7052 134.62 0)
 			(hide yes)
@@
 			)
 		)
-		(property "Footprint" ""
+		(property "Footprint" "Capacitor_SMD:C_0603_1608Metric_Pad1.08x0.95mm_HandSolder"
 			(at 36.5252 134.62 0)
 			(hide yes)
@@
 			)
 		)
-		(property "Footprint" ""
+		(property "Footprint" "Capacitor_SMD:C_1206_3216Metric_Pad1.33x1.80mm_HandSolder"
 			(at 120.3452 57.15 0)
 			(hide yes)
@@
 			)
 		)
-		(property "Footprint" ""
+		(property "Footprint" "Capacitor_SMD:C_0603_1608Metric_Pad1.08x0.95mm_HandSolder"
 			(at 134.3152 118.11 0)
 			(hide yes)
@@
 			)
 		)
-		(property "Footprint" ""
+		(property "Footprint" "Resistor_SMD:R_0603_1608Metric_Pad0.98x0.95mm_HandSolder"
 			(at 251.206 58.674 90)
 			(hide yes)
@@
 			)
 		)
-		(property "Footprint" "rov_power:SOT-23-5_MC_MCH"
+		(property "Footprint" "Capacitor_SMD:C_0603_1608Metric_Pad1.08x0.95mm_HandSolder"
 			(at 84.7852 48.26 0)
 			(hide yes)
@@
 			)
 		)
-		(property "Footprint" ""
+		(property "Footprint" "Resistor_SMD:R_0603_1608Metric_Pad0.98x0.95mm_HandSolder"
 			(at 50.546 106.426 90)
 			(hide yes)
@@
 			)
 		)
-		(property "Footprint" ""
+		(property "Footprint" "Capacitor_SMD:C_1206_3216Metric_Pad1.33x1.80mm_HandSolder"
 			(at 154.6352 57.15 0)
 			(hide yes)
@@
 			)
 		)
-		(property "Footprint" "rov_power:SOT-23-5_MC_MCH"
+		(property "Footprint" "Capacitor_SMD:C_0603_1608Metric_Pad1.08x0.95mm_HandSolder"
 			(at 27.6352 46.99 0)
 			(hide yes)
@@
 			)
 		)
-		(property "Footprint" ""
+		(property "Footprint" "Capacitor_SMD:C_1206_3216Metric_Pad1.33x1.80mm_HandSolder"
 			(at 143.2052 57.15 0)
 			(hide yes)
@@
 			)
 		)
-		(property "Footprint" ""
+		(property "Footprint" "TestPoint:TestPoint_Pad_D4.0mm"
 			(at 194.31 120.65 0)
 			(hide yes)
@@
 			)
 		)
-		(property "Footprint" ""
+		(property "Footprint" "Capacitor_SMD:C_0603_1608Metric_Pad1.08x0.95mm_HandSolder"
 			(at 145.7452 118.11 0)
 			(hide yes)
@@
 			)
 		)
-		(property "Footprint" ""
+		(property "Footprint" "Resistor_SMD:R_0603_1608Metric_Pad0.98x0.95mm_HandSolder"
 			(at 241.046 58.674 90)
 			(hide yes)
@@
 			)
 		)
-		(property "Footprint" ""
+		(property "Footprint" "Resistor_SMD:R_0603_1608Metric_Pad0.98x0.95mm_HandSolder"
 			(at 241.046 155.194 90)
 			(hide yes)
@@
 			)
 		)
-		(property "Footprint" ""
+		(property "Footprint" "TestPoint:TestPoint_Pad_D4.0mm"
 			(at 194.31 57.15 0)
 			(hide yes)
@@
 			)
 		)
-		(property "Footprint" ""
+		(property "Footprint" "Resistor_SMD:R_0603_1608Metric_Pad0.98x0.95mm_HandSolder"
 			(at 251.206 122.174 90)
 			(hide yes)
@@
 			)
 		)
-		(property "Footprint" ""
+		(property "Footprint" "TestPoint:TestPoint_Pad_D4.0mm"
 			(at 194.31 87.63 0)
 			(hide yes)
@@
 			)
 		)
-		(property "Footprint" ""
+		(property "Footprint" "Resistor_SMD:R_0603_1608Metric_Pad0.98x0.95mm_HandSolder"
 			(at 241.046 89.154 90)
 			(hide yes)
@@
 			)
 		)
-		(property "Footprint" ""
+		(property "Footprint" "Capacitor_SMD:C_1206_3216Metric_Pad1.33x1.80mm_HandSolder"
 			(at 131.7752 57.15 0)
 			(hide yes)
@@
 			)
 		)
-		(property "Footprint" ""
+		(property "Footprint" "Capacitor_SMD:C_0603_1608Metric_Pad1.08x0.95mm_HandSolder"
 			(at 122.8852 118.11 0)
 			(hide yes)
@@
 			)
 		)
-		(property "Footprint" ""
+		(property "Footprint" "Resistor_SMD:R_0603_1608Metric_Pad0.98x0.95mm_HandSolder"
 			(at 251.206 89.154 90)
 			(hide yes)
@@
 			)
 		)
-		(property "Footprint" ""
+		(property "Footprint" "Resistor_SMD:R_0603_1608Metric_Pad0.98x0.95mm_HandSolder"
 			(at 251.206 155.194 90)
 			(hide yes)

Commit message: office hour changes
Parts:
- C16, C22, C24, C25, C28, C29, C30, C34, C35, C36, C39, C40, C41: footprint (none) -> Capacitor_THT:CP_Radial_D10.0mm_P5.00mm
- C23, C27, C32, C37: footprint Capacitor_SMD:C_1206_3216Metric_Pad1.33x1.80mm_HandSolder -> Capacitor_SMD:C_0805_2012Metric_Pad1.18x1.45mm_HandSolder
- C26, C31, C33, C38: footprint Capacitor_SMD:C_0603_1608Metric_Pad1.08x0.95mm_HandSolder -> Capacitor_SMD:C_0805_2012Metric_Pad1.18x1.45mm_HandSolder
- PG1, PG2, PG3, PG4: footprint TestPoint:TestPoint_Pad_D4.0mm -> TestPoint:TestPoint_Pad_D2.5mm
- U7: footprint i6A4W_DIP_FULL_TDK -> i6A4W_DIP_FULL_TDK.kicad_mod:i6A4W_DIP_FULL_TDK
Other:
- note removed: "63V 1206 caps"
Changed lines of the file:
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@@
 		)
 	)
-	(text "63V 1206 caps"
-		(exclude_from_sim no)
-		(at 165.1 58.674 0)
-		(effects
-			(font
-				(size 1.27 1.27)
-				(color 255 0 23 1)
-			)
-		)
-	)
 	(text "I2C Address: \n0x20 (Hex)"
 		(exclude_from_sim no)
@@
 			)
 		)
-		(property "Footprint" "Capacitor_SMD:C_0603_1608Metric_Pad1.08x0.95mm_HandSolder"
+		(property "Footprint" "Capacitor_SMD:C_0805_2012Metric_Pad1.18x1.45mm_HandSolder"
 			(at 157.1752 118.11 0)
 			(hide yes)
@@
 			)
 		)
-		(property "Footprint" ""
+		(property "Footprint" "Capacitor_THT:CP_Radial_D10.0mm_P5.00mm"
 			(at 162.2552 77.47 0)
 			(hide yes)
@@
 			)
 		)
-		(property "Footprint" ""
+		(property "Footprint" "Capacitor_THT:CP_Radial_D10.0mm_P5.00mm"
 			(at 150.8252 97.79 0)
 			(hide yes)
@@
 			)
 		)
-		(property "Footprint" "TestPoint:TestPoint_Pad_D4.0mm"
+		(property "Footprint" "TestPoint:TestPoint_Pad_D2.5mm"
 			(at 194.31 153.67 0)
 			(hide yes)
@@
 			)
 		)
-		(property "Footprint" ""
+		(property "Footprint" "Capacitor_THT:CP_Radial_D10.0mm_P5.00mm"
 			(at 23.8252 134.62 0)
 			(hide yes)
@@
 			)
 		)
-		(property "Footprint" ""
+		(property "Footprint" "Capacitor_THT:CP_Radial_D10.0mm_P5.00mm"
 			(at 131.7752 77.47 0)
 			(hide yes)
@@
 			)
 		)
-		(property "Footprint" ""
+		(property "Footprint" "Capacitor_THT:CP_Radial_D10.0mm_P5.00mm"
 			(at 120.3452 97.79 0)
 			(hide yes)
@@
 			)
 		)
-		(property "Footprint" "Capacitor_SMD:C_1206_3216Metric_Pad1.33x1.80mm_HandSolder"
+		(property "Footprint" "Capacitor_SMD:C_0805_2012Metric_Pad1.18x1.45mm_HandSolder"
 			(at 120.3452 57.15 0)
 			(hide yes)
@@
 			)
 		)
-		(property "Footprint" ""
+		(property "Footprint" "Capacitor_THT:CP_Radial_D10.0mm_P5.00mm"
 			(at 150.8252 77.47 0)
 			(hide yes)
@@
 			)
 		)
-		(property "Footprint" ""
+		(property "Footprint" "Capacitor_THT:CP_Radial_D10.0mm_P5.00mm"
 			(at 120.3452 38.1 0)
 			(hide yes)
@@
 			)
 		)
-		(property "Footprint" "Capacitor_SMD:C_0603_1608Metric_Pad1.08x0.95mm_HandSolder"
+		(property "Footprint" "Capacitor_SMD:C_0805_2012Metric_Pad1.18x1.45mm_HandSolder"
 			(at 134.3152 118.11 0)
 			(hide yes)
@@
 			)
 		)
-		(property "Footprint" ""
+		(property "Footprint" "Capacitor_THT:CP_Radial_D10.0mm_P5.00mm"
 			(at 162.2552 38.1 0)
 			(hide yes)
@@
 			)
 		)
-		(property "Footprint" ""
+		(property "Footprint" "Capacitor_THT:CP_Radial_D10.0mm_P5.00mm"
 			(at 134.3152 38.1 0)
 			(hide yes)
@@
 			)
 		)
-		(property "Footprint" "Capacitor_SMD:C_1206_3216Metric_Pad1.33x1.80mm_HandSolder"
+		(property "Footprint" "Capacitor_SMD:C_0805_2012Metric_Pad1.18x1.45mm_HandSolder"
 			(at 154.6352 57.15 0)
 			(hide yes)
@@
 			)
 		)
-		(property "Footprint" "Capacitor_SMD:C_1206_3216Metric_Pad1.33x1.80mm_HandSolder"
+		(property "Footprint" "Capacitor_SMD:C_0805_2012Metric_Pad1.18x1.45mm_HandSolder"
 			(at 143.2052 57.15 0)
 			(hide yes)
@@
 			)
 		)
-		(property "Footprint" "TestPoint:TestPoint_Pad_D4.0mm"
+		(property "Footprint" "TestPoint:TestPoint_Pad_D2.5mm"
 			(at 194.31 120.65 0)
 			(hide yes)
@@
 			)
 		)
-		(property "Footprint" "Capacitor_SMD:C_0603_1608Metric_Pad1.08x0.95mm_HandSolder"
+		(property "Footprint" "Capacitor_SMD:C_0805_2012Metric_Pad1.18x1.45mm_HandSolder"
 			(at 145.7452 118.11 0)
 			(hide yes)
@@
 			)
 		)
-		(property "Footprint" ""
+		(property "Footprint" "Capacitor_THT:CP_Radial_D10.0mm_P5.00mm"
 			(at 162.2552 97.79 0)
 			(hide yes)
@@
 			)
 		)
-		(property "Footprint" "TestPoint:TestPoint_Pad_D4.0mm"
+		(property "Footprint" "TestPoint:TestPoint_Pad_D2.5mm"
 			(at 194.31 57.15 0)
 			(hide yes)
@@
 			)
 		)
-		(property "Footprint" "i6A4W_DIP_FULL_TDK"
+		(property "Footprint" "i6A4W_DIP_FULL_TDK.kicad_mod:i6A4W_DIP_FULL_TDK"
 			(at 24.13 83.82 0)
 			(hide yes)
@@
 			)
 		)
-		(property "Footprint" "TestPoint:TestPoint_Pad_D4.0mm"
+		(property "Footprint" "TestPoint:TestPoint_Pad_D2.5mm"
 			(at 194.31 87.63 0)
 			(hide yes)
@@
 			)
 		)
-		(property "Footprint" ""
+		(property "Footprint" "Capacitor_THT:CP_Radial_D10.0mm_P5.00mm"
 			(at 148.2852 38.1 0)
 			(hide yes)
@@
 			)
 		)
-		(property "Footprint" ""
+		(property "Footprint" "Capacitor_THT:CP_Radial_D10.0mm_P5.00mm"
 			(at 120.3452 77.47 0)
 			(hide yes)
@@
 			)
 		)
-		(property "Footprint" "Capacitor_SMD:C_1206_3216Metric_Pad1.33x1.80mm_HandSolder"
+		(property "Footprint" "Capacitor_SMD:C_0805_2012Metric_Pad1.18x1.45mm_HandSolder"
 			(at 131.7752 57.15 0)
 			(hide yes)
@@
 			)
 		)
-		(property "Footprint" "Capacitor_SMD:C_0603_1608Metric_Pad1.08x0.95mm_HandSolder"
+		(property "Footprint" "Capacitor_SMD:C_0805_2012Metric_Pad1.18x1.45mm_HandSolder"
 			(at 122.8852 118.11 0)
 			(hide yes)
@@
 			)
 		)
-		(property "Footprint" ""
+		(property "Footprint" "Capacitor_THT:CP_Radial_D10.0mm_P5.00mm"
 			(at 131.7752 97.79 0)
 			(hide yes)
